File: qualification/class-b/usb-uart/kicad/usb_uart.kicad_sch (KiCad schematic)
At the start: 36 parts, among them J1 TYPE-C-31-M-12, J2 UART1, J3 FLOW1, J4 RS485, U1 CH342F, U2 LDO, U3 THVD1450D

Commit message: SYN-66 - Keep a net name label off the wires of other nets
Signed-off-by: nyagamunene <stevenyaga2014@gmail.com>
Connections:
- net RXD1_MCU: no longer R8.2, U1.1 (ri0), U1.14 (dsr1_tnow1), U1.16 (dcd1), U1.17 (ri1), U1.22 (dsr0), U1.24 (dcd0)
- new net MODEM_IDLE: R8.2, U1.1 (ri0), U1.14 (dsr1_tnow1), U1.16 (dcd1), U1.17 (ri1), U1.22 (dsr0), U1.24 (dcd0)
Changed lines of the file:
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@@
 	(label
 		"MODEM_IDLE"
-		(at 242.57 49.53 0)
+		(at 242.57 48.26 0)
 		(effects
 			(font

Commit message: SYN-66 - Re-export and re-route the board with the TX LED fix and clean silkscreen
Signed-off-by: nyagamunene <stevenyaga2014@gmail.com>
Connections:
- net GND: no longer D4.1 (K), D7.1 (K)
- net TXD0: now also D4.1 (K); no longer R4.1
- net TXD1: now also D7.1 (K); no longer R7.1
- net VIO: now also R4.1, R7.1
Other:
- note added: "D4/D7 red LEDs from VIO, sunk into TXD0/TXD1: dark while the line idles, lit on the low bits."
- note removed: "D4/D7 red LEDs from TXD0/TXD1."
- moved on the sheet: C2, C3, C4, C5, C6, C7, D1, D2, D3, D4, D5, D6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

Commit message: SYN-66 - Regenerate the usb-uart schematic and ERC with the VIO power flag
ERC now reports 0 errors. The PCB is unchanged.

Signed-off-by: nyagamunene <stevenyaga2014@gmail.com>
Changed lines of the file:
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@@
+	(symbol
+		(lib_id "power:PWR_FLAG")
+		(at 309.88 175.26 0)
+		(unit 1)
+		(in_bom no)
+		(on_board no)
+		(property
+			"Reference"
+			"#FLG3022"
+			(at 309.88 175.26 0)
+			(effects
+				(font
+					(size 1.27 1.27)
+				)
+				(hide yes)
+			)
+		)
+		(property
+			"Value"
+			"PWR_FLAG"
+			(at 309.88 175.26 0)
+			(effects
+				(font
+					(size 1.27 1.27)
+				)
+				(hide yes)
+			)
+		)
+	)
 	(symbol
 		(lib_id "power:PWR_FLAG")
