File: qualification/class-b/buck/kicad/buck.kicad_sch (KiCad schematic)
At the start: 20 parts, among them J1 24V_IN, J2 3V3_OUT, U1 TPS54202DDCR

Commit message: SYN-67 - Re-export the buck board on current main and give it its own case
Re-ran the whole chain on main 1eac8a1 (KiCad 10.0.7, FreeRouting 2.4.1,
OpenJDK 25.0.5). The exporter's 1.5 mm edge rim (#272) shrinks the outline
from 63.0 x 37.6 mm to 58.0 x 32.6 mm; every part position is unchanged,
and three export runs gave byte-identical KiCad files.

Adds the manufacturing exports #38 asks for: 22 Gerbers plus the job file,
PTH and NPTH drill files, and pick-and-place. Adds a second release report,
because asking for the fab package flips the same board from release_ready
true to untrusted on the 7 unreviewed parts; both answers are kept.

QUALIFICATION.md is rewritten around this board instead of a shared
template: the A rows are the measurements above, the B rows name the
capability-descriptor limits they rest on (thermal_relief_analysis,
power_sequencing_and_power_good, split_ground_planes,
return_path_and_layer_transition_analysis), and a new section maps every
#38 "Check exactly" line to a verdict for this board. It also carries the
[[board]] row this board declares for qualification/matrix.toml, with no
expect value invented: synth check cannot select FreeRouting at this
revision and no KiCadRoutingTools checkout was available to measure it.

Also corrects stale claims: the negative twin has 13 warnings not 14, the
schematic's net names now match the PCB, and the MCP placement review
passes (score 100) instead of reporting a stale outline.

Signed-off-by: nyagamunene <stevenyaga2014@gmail.com>
Connections:
- net VIN_RAW: now reaches F1.1, J1.1 (Pin_1)
- net BOOT: now reaches C4.1, U1.6 (BOOT)
- net VIN_FUSED: now reaches D1.2 (A), F1.2
- net P2 renamed +3V3
- net P2_R_LED renamed LED_PWR
Other:
- moved on the sheet: C1, C2, C3, C4, C5, C6, C7, D1, D2, D3, F1, J1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

Commit message: SYN-67 - Rebuild the buck board around it and re-prove the A rows
25 components including two M2.5 mounting holes, a 4-pin output connector
(+3V3, GND, PG, GND) and the values from LMR33640 Table 9-2: 6.8 uH, 3x
22 uF out, 10 uF + 220 nF in, 1 uF VCC, 100 nF boot, 100k/43.2k feedback,
56 pF feed-forward, 1.37M/100k UVLO (18.1 V / 16.6 V). PG is open drain and
pulled up through 100k.

Re-routed with FreeRouting 2.4.1 on main 1eac8a1: 12 nets, 0 open, 81
segments, 18 vias, 0 blocking findings. Outline 71.9 x 31.1 mm. KiCad DRC
0/0/30 (5 are silkscreen, new with the denser placement), ERC 0/68. Two
exports byte-identical; gerbers, drill, BOM, pick-and-place and images
regenerated; 50 hashes rewritten.

QUALIFICATION.md now proves the power-good net and the thermal pad (A15,
A16) and keeps their behaviour unverified (B3, B2). The overvoltage row is
bounded honestly: a sustained 28-32 V rail is inside the 36 V rating, a
surge is not covered because the TVS clamps above the 38 V absolute max.

Signed-off-by: nyagamunene <stevenyaga2014@gmail.com>
Parts:
- added C8: 1uF, Capacitor_SMD:C_0603_1608Metric, symbol Device:C
- added C9: 22uF, Capacitor_SMD:C_1206_3216Metric, symbol Device:C
- added H1, H2: M2.5, MountingHole:MountingHole_2.5mm, symbol Mechanical:MountingHole
- added R_PG: 100k, Resistor_SMD:R_0603_1608Metric, symbol Device:R_US
- C3: value 100nF -> 220nF
- D2: value SMBJ26A -> SMBJ30A; MPN SMBJ26A -> SMBJ30A
- J2: footprint Connector_JST:JST_XH_B2B-XH-A_1x02_P2.50mm_Vertical -> Connector_JST:JST_XH_B4B-XH-A_1x04_P2.50mm_Vertical; symbol Connector_Generic:Conn_01x02 -> Connector_Generic:Conn_01x04; MPN B2B-XH-A -> B4B-XH-A
- L1: value 10uH -> 6.8uH; MPN SRN6045TA-100M -> SRN6045TA-6R8M
- R_FB_B: value 22.1k -> 43.2k
- R_UV_T: value 1.5M -> 1.37M
- U1: value TPS54202DDCR -> LMR33640ADDA; footprint Package_TO_SOT_SMD:SOT-23-6 -> Package_SO:HSOP-8-1EP_3.9x4.9mm_P1.27mm_EP2.41x3.1mm; symbol Regulator_Switching:TPS54202DDC -> Regulator_Switching:LMR33640ADDA; MPN TPS54202DDCR -> LMR33640ADDA
Connections:
- net +3V3: now also C9.1, R_PG.2
- net BOOT: now also U1.7 (BOOT); no longer U1.6 (BOOT)
- net EN: now also U1.3 (EN); no longer U1.5 (EN)
- net FB: now also U1.5 (FB); no longer U1.4 (FB)
- net GND: now also J2.4 (Pin_4), U1.9 (GND), C8.2, C9.2
- net SW: now also U1.8 (SW); no longer U1.2 (SW)
- net VIN: now also U1.2 (VIN); no longer U1.3 (VIN)
- new net PG: J2.3 (Pin_3), R_PG.1, U1.4 (PG)
- new net U1_VCC: C8.1, U1.6 (VCC)
Other:
- note added: "50 V parts for a 24 V rail; DC-bias derating of C2 is not known."
- note added: "C1 bulk, C2 ceramic, C3 high-frequency next to the VIN pin (LMR33640 Table 9-2: 10 uF + 220 nF)."
- note added: "C4 100 nF boot capacitor between BOOT and SW; C8 1 uF on VCC."
- note added: "C7 56 pF feed-forward across the upper resistor (datasheet Eq 9 gives about 60 pF)."
- note added: "D2 TVS (30 V standoff) sits after D1, directly on the VIN node. It clamps ESD and transient energy only; the clamp is above U1's absolute maximum, so it is not an OVP."
- note added: "EN divider from VIN. LMR33640 VEN-H 1.231 V typical, 100 mV hysteresis: start 18.1 V, stop 16.6 V."
- note added: "EN stays under 2 V at a 28 V input (EN absolute maximum is VIN + 0.3 V)."
- note added: "J2 pin 1 is +3.3 V, pin 2 GND, pin 3 power-good (3.3 V logic, 100k pull-up), pin 4 GND."
- note added: "L1 6.8 uH and 3x 22 uF follow Table 9-2 for 3.3 V at 400 kHz (minimum Cout is 3x 22 uF)."
- note added: "LMR33640: 400 kHz, internal compensation, exposed pad (pin 9) on GND, open-drain PG."
- note added: "MECHANICAL"
- note added: "PG goes low during start-up and on a fault, so J2 pin 3 reads valid only after the 4 ms start-up delay."
- note added: "PG is open drain and pulled up to +3V3 through 100k (datasheet 8.3.1 suggests 100k to VCC or VOUT)."
- note added: "POWER GOOD"
- note added: "The exposed pad (pin 9) is soldered to the F.Cu GND pour. There are no vias in the pad:"
- note added: "Two M2.5 non-plated holes in opposite corners; the board is fixed down through them."
- note added: "Vout = 1.0 V x (1 + 100k / 43.2k) = 3.31 V."
- note added: "the board's fabrication floor is a 0.3 mm drill and the KiCad thermal-via footprint ships 0.2 mm."
- note removed: "50 V parts for a 24 V rail; DC-bias derating not known, effective C2 may be under 10 uF."
- note removed: "C1 bulk, C2 ceramic (datasheet: over 10 uF), C3 high-frequency next to the VIN pin."
- note removed: "C4 100 nF boot capacitor between BOOT and SW."
- note removed: "C5/C6 are 25 V X7R; DC-bias derating unknown. fo = 3.95/(Vout x COUT) must stay under 40 kHz."
- note removed: "C7 56 pF feed-forward across the upper resistor (Table 7-2)."
- note removed: "D2 TVS (26 V standoff) sits after D1, directly on the VIN node. It clamps surge energy only."
- note removed: "EN divider from VIN. Datasheet Eq 1 and 2 give start 18.31 V, stop 15.67 V (typical thresholds)."
- note removed: "EN stays under 1.75 V at a 28 V input (EN limit 5.5 V)."
- note removed: "J2 pin 1 is +3.3 V, pin 2 is GND."
- note removed: "L1 10 uH and 2x 22 uF follow datasheet Table 7-2 for 3.3 V (44 uF)."
- note removed: "TPS54202: 500 kHz, internal compensation, no power-good pin."
- note removed: "Vout = 0.596 V x (1 + 100k / 22.1k) = 3.29 V."
- note removed: "With 1% resistors: start 17.96-18.67 V, stop 15.35-15.99 V."
- moved on the sheet: C1, C2, C3, C4, C5, C6, C7, D1, D2, D3, F1, L1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

Commit message: SYN-67 - Add a power-good fault LED to the buck board
D4 and R_PGLED run from +3V3 to PG, so the LED lights while the open-drain PG pin is low. Reuses the existing ltst_c190kgkt part, no registry change. Adding the two parts re-ran the router, so the KiCad files, reports, renders and hashes are regenerated and the docs carry the new numbers (13 nets, 27 parts, 16 GND vias).

Signed-off-by: nyagamunene <stevenyaga2014@gmail.com>
Parts:
- added D4: PG FAULT, LED_SMD:LED_0603_1608Metric, symbol Device:LED
- added R_PGLED: 470, Resistor_SMD:R_0603_1608Metric, symbol Device:R_US
Connections:
- net +3V3: now also R_PGLED.1
- net PG: now also D4.1 (K)
- new net LED_PG: D4.2 (A), R_PGLED.2
Other:
- note added: "About 2.5 mA when lit (470 R, Vf about 2.1 V); U1's PG pull-down is 76 to 150 ohm RDSON, so PG stays near 0.4 V."
- note added: "D4 green fault LED from +3V3 through R_PGLED to PG: it is lit while PG is low, dark while power is good."
- moved on the sheet: C1, C2, C3, C4, C5, C6, C7, C8, C9, D1, D2, D3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

Commit message: SYN-67 - Place the buck board with Synth's own placer and regenerate the evidence on one head
Signed-off-by: nyagamunene <stevenyaga2014@gmail.com>
Parts:
- C1: MPN (none) -> RVT1H470M0810
Changed lines of the file:
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@@
 		(property
 			"Datasheet"
-			""
+			"https://wmsc.lcsc.com/wmsc/upload/file/pdf/v2/lcsc/2109290630_Honor-Elec-RVT1H470M0810_C2895739.pdf"
 			(at 27.94 116.84 0)
 			(effects
@@
 		(property
 			"MPN"
-			""
+			"RVT1H470M0810"
 			(at 27.94 116.84 0)
 			(effects

Commit message: SYN-67 - Regenerate the buck artifacts and rewrite the evidence for the LMR38010 board, add the matrix row
Signed-off-by: nyagamunene <stevenyaga2014@gmail.com>
Parts:
- removed C8: 1uF, Capacitor_SMD:C_0603_1608Metric, symbol Device:C
- added R_RT: 33k, Resistor_SMD:R_0603_1608Metric, symbol Device:R_US
- D1: symbol Diode:SS36 -> Device:D_Schottky
- U1: value LMR33640ADDA -> LMR38010SDDAR; symbol Regulator_Switching:LMR33640ADDA -> synth:lmr38010; MPN LMR33640ADDA -> LMR38010SDDAR
Connections:
- net U1_VCC is gone; now on net PG: U1.6 (pg)
- net EN: now also U1.2 (en); no longer U1.3 (EN)
- net GND: now also R_RT.2
- net PG: no longer U1.4 (PG)
- net VIN: now also U1.3 (vin); no longer U1.2 (VIN)
- new net RT: R_RT.1, U1.4 (rt_sync)
Other:
- note added: "About 2.5 mA when lit (470 R, Vf about 2.1 V); U1's PG pull-down is about 92 ohm RDSON, so PG stays near 0.4 V."
- note added: "C1 bulk, C2 ceramic, C3 high-frequency next to the VIN pin (LMR38010 section 9.2.2.6: at least 4.7 uF + 100 to 220 nF)."
- note added: "C4 100 nF boot capacitor between BOOT and SW."
- note added: "D2 TVS (30 V standoff) sits after D1, directly on the VIN node. Its 48.4 V clamp is below U1's 85 V absolute maximum, so U1 stays within its rating under a surge the TVS can absorb."
- note added: "EN divider from VIN. LMR38010 VEN-H 1.25 V typical (1.1 to 1.4), VEN-L 1.10 V typical: start 18.4 V (16.2 to 20.6 V), stop 16.2 V."
- note added: "L1 6.8 uH at 800 kHz gives about 0.5 A ripple at 26.4 V in (datasheet Eq 10 K about 0.5), above the 1.03 uH minimum of Eq 11 (0.25 x 3.3 V / 800 kHz); 3x 22 uF is unverified: Table 9-1 has no 3.3 V row."
- note added: "LMR38010SDDAR: internal compensation, exposed pad (pin 9) on GND, open-drain PG, PFM with spread spectrum."
- note added: "PG is open drain and pulled up to +3V3 through 100k (datasheet 8.3.5: pull up through a resistor; PG tolerates 20 V)."
- note added: "R_RT 33k from RT/SYNC to GND sets 800 kHz (RT table under datasheet Figure 8-4); the pin must not float."
- note removed: "About 2.5 mA when lit (470 R, Vf about 2.1 V); U1's PG pull-down is 76 to 150 ohm RDSON, so PG stays near 0.4 V."
- note removed: "C1 bulk, C2 ceramic, C3 high-frequency next to the VIN pin (LMR33640 Table 9-2: 10 uF + 220 nF)."
- note removed: "C4 100 nF boot capacitor between BOOT and SW; C8 1 uF on VCC."
- note removed: "D2 TVS (30 V standoff) sits after D1, directly on the VIN node. It clamps ESD and transient energy only; the clamp is above U1's absolute maximum, so it is not an OVP."
- note removed: "EN divider from VIN. LMR33640 VEN-H 1.231 V typical, 100 mV hysteresis: start 18.1 V, stop 16.6 V."
- note removed: "L1 6.8 uH and 3x 22 uF follow Table 9-2 for 3.3 V at 400 kHz (minimum Cout is 3x 22 uF)."
- note removed: "LMR33640: 400 kHz, internal compensation, exposed pad (pin 9) on GND, open-drain PG."
- note removed: "PG is open drain and pulled up to +3V3 through 100k (datasheet 8.3.1 suggests 100k to VCC or VOUT)."
- moved on the sheet: C1, C2, C3, C4, C5, C6, C7, C9, D3, D4, J2, L1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
