File: qualification/class-a/irrigation-controller/export/irrigation_controller.kicad_sch (KiCad schematic)
At the start: 126 parts, among them J1 (no value), Q1 AO3401A, U1 MP2307DN-LF-Z, U2 (no value), U4 (no value), U5 (no value), Y1 NX3225GD-8MHZ-STD-CRA-3

Commit message: qualification(irrigation): the schematic carries a power flag on +12V_VALVE; ERC reports no error
The exported schematic and the ERC report come from three fresh exports made with
Synth f7b110db; the routed board, the Gerbers, the BOM and the placement file are
unchanged (masked board hash ef9c39148e, Gerber hash 125847925c).
Changed lines of the file:
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@@
+	(symbol
+		(lib_id "power:PWR_FLAG")
+		(at 119.38 59.69 0)
+		(unit 1)
+		(in_bom no)
+		(on_board no)
+		(property
+			"Reference"
+			"#FLG4729"
+			(at 119.38 59.69 0)
+			(effects
+				(font
+					(size 1.27 1.27)
+				)
+				(hide yes)
+			)
+		)
+		(property
+			"Value"
+			"PWR_FLAG"
+			(at 119.38 59.69 0)
+			(effects
+				(font
+					(size 1.27 1.27)
+				)
+				(hide yes)
+			)
+		)
+	)
 	(symbol
 		(lib_id "power:PWR_FLAG")
